Commit message: tf

File: dji_description/urdf/dji.xacro (robot description, xacro)
@@ -65,5 +65,5 @@
   </link>
   <joint name="camera_joint" type="fixed">
-    <axis xyz="1 0 0" />
+    <axis xyz="0 0 1" />
     <origin xyz="0.18 0 0.2" rpy="0 0 0"/>
     <parent link="dji_link"/>

Commit message: gimbal control

File: dji_description/urdf/dji.xacro (robot description, xacro)
@@ -64,5 +64,5 @@
     </inertial>
   </link>
-  <joint name="camera_joint" type="fixed">
+  <joint name="camera_joint" type="continuous">
     <axis xyz="0 0 1" />
     <origin xyz="0.18 0 0.2" rpy="0 0 0"/>
@@ -102,3 +102,13 @@
     </actuator>
   </transmission>
+  <transmission name="tran2">
+    <type>transmission_interface/SimpleTransmission</type>
+    <joint name="camera_joint">
+      <hardwareInterface>EffortJointInterface</hardwareInterface>
+    </joint>
+    <actuator name="camera_motor">
+      <hardwareInterface>EffortJointInterface</hardwareInterface>
+      <mechanicalReduction>1</mechanicalReduction>
+    </actuator>
+  </transmission>
 </robot>

Commit message: adding robot city bridge world

File: dji_description/urdf/dji.xacro (robot description, xacro)
@@ -5,6 +5,6 @@
   <xacro:property name="PI" value="3.1415926535897931"/>
   <xacro:property name="mass" value="30" /> <!-- arbitrary value for mass -->
-  <xacro:property name="width" value="0.3" /> <!-- Square dimensions (widthxwidth) of beams -->
-  <xacro:property name="height" value="0.3" /> <!-- DJI height -->
+  <xacro:property name="width" value="1.0" /> <!-- Square dimensions (widthxwidth) of beams -->
+  <xacro:property name="height" value="1.0" /> <!-- DJI height -->
   <!-- Import all Gazebo-customization elements, including Gazebo colors -->
   <xacro:include filename="$(find dji_description)/urdf/dji.gazebo" />
@@ -13,5 +13,5 @@
   <!-- DJI Body Link -->
   <link name="dji_link">
-    <collision>
+    <collision name="dji_body_collision">
       <origin xyz="0 0 ${height/2}" rpy="0 0 0"/>
       <geometry>
@@ -35,4 +35,10 @@
 	  izz="${mass / 12.0 * (width*width + width*width)}"/>
     </inertial>
+<!--
+    <sensor name='dji_body_collision' type='contact'>
+      <contact>
+        <collision>collision</collision>
+      </contact>
+    </sensor> -->
   </link>
   <joint name="hokuyo_joint" type="continuous">

Commit message: working with gym-gazebo. Added state publisher to g2_control to publish state from laser data.

File: dji_description/urdf/dji.xacro (robot description, xacro)
@@ -5,6 +5,6 @@
   <xacro:property name="PI" value="3.1415926535897931"/>
   <xacro:property name="mass" value="30" /> <!-- arbitrary value for mass -->
-  <xacro:property name="width" value="1.0" /> <!-- Square dimensions (widthxwidth) of beams -->
-  <xacro:property name="height" value="1.0" /> <!-- DJI height -->
+  <xacro:property name="width" value="0.1" /> <!-- Square dimensions (widthxwidth) of beams -->
+  <xacro:property name="height" value="0.4" /> <!-- DJI height -->
   <!-- Import all Gazebo-customization elements, including Gazebo colors -->
   <xacro:include filename="$(find dji_description)/urdf/dji.gazebo" />
@@ -13,10 +13,10 @@
   <!-- DJI Body Link -->
   <link name="dji_link">
-    <collision name="dji_body_collision">
-      <origin xyz="0 0 ${height/2}" rpy="0 0 0"/>
-      <geometry>
-	    <box size="${width} ${width} ${height}"/>
-      </geometry>
-    </collision>
+    <!-- <collision name="dji_body_collision"> -->
+      <!-- <origin xyz="0 0 ${height/2}" rpy="0 0 0"/> -->
+      <!-- <geometry> -->
+          <!-- <sphere radius ="1.25" /> -->
+      <!-- </geometry> -->
+    <!-- </collision>  -->
     <visual>
       <origin xyz="0 0 0" rpy="0 0 0"/>
@@ -35,10 +35,4 @@
 	  izz="${mass / 12.0 * (width*width + width*width)}"/>
     </inertial>
-<!--
-    <sensor name='dji_body_collision' type='contact'>
-      <contact>
-        <collision>collision</collision>
-      </contact>
-    </sensor> -->
   </link>
   <joint name="hokuyo_joint" type="continuous">
@@ -50,9 +44,9 @@
   </joint>
   <!-- Hokuyo Laser -->
-  <link name="hokuyo_link">
+  <link name="hokuyo_link" selfCollide="false">
     <collision>
       <origin xyz="0 0 0.0" rpy="0 0 0"/>
       <geometry>
-	    <box size="0.1 0.1 0.1"/>
+          <sphere radius ="1.25" />
       </geometry>
     </collision>
@@ -70,32 +64,4 @@
     </inertial>
   </link>
-  <joint name="camera_joint" type="continuous">
-    <axis xyz="0 0 1" />
-    <origin xyz="0.18 0 0.2" rpy="0 0 0"/>
-    <parent link="dji_link"/>
-    <child link="camera_link"/>
-  </joint>
-  <!-- Camera -->
-  <link name="camera_link">
-    <collision>
-      <origin xyz="0 0 0" rpy="0 0 0"/>
-      <geometry>
-	<box size="0.03 0.02 0.02"/>
-      </geometry>
-    </collision>
-    <visual>
-      <origin xyz="0 0 0" rpy="0 0 0 "/>
-      <geometry>
-	    <box size="0.06 0.03 0.03"/>
-	    <!-- <cylinder length="0.06" radius="0.02"/> -->
-      </geometry>
-      <material name="white"/>
-    </visual>
-    <inertial>
-      <mass value="1e-5" />
-      <origin xyz="0 0 0" rpy="0 0 0"/>
-      <inertia ixx="1e-6" ixy="0" ixz="0" iyy="1e-6" iyz="0" izz="1e-6" />
-    </inertial>
-  </link>
   <transmission name="tran1">
     <type>transmission_interface/SimpleTransmission</type>
@@ -108,13 +74,3 @@
     </actuator>
   </transmission>
-  <transmission name="tran2">
-    <type>transmission_interface/SimpleTransmission</type>
-    <joint name="camera_joint">
-      <hardwareInterface>EffortJointInterface</hardwareInterface>
-    </joint>
-    <actuator name="camera_motor">
-      <hardwareInterface>EffortJointInterface</hardwareInterface>
-      <mechanicalReduction>1</mechanicalReduction>
-    </actuator>
-  </transmission>
 </robot>

Commit message: creating accel_sim_branch

File: dji_description/urdf/dji.xacro (robot description, xacro)
@@ -6,5 +6,5 @@
   <xacro:property name="mass" value="30" /> <!-- arbitrary value for mass -->
   <xacro:property name="width" value="1.0" /> <!-- Square dimensions (widthxwidth) of beams -->
-  <xacro:property name="height" value="1.0" /> <!-- DJI height -->
+  <xacro:property name="height" value="0.5" /> <!-- DJI height -->
   <!-- Import all Gazebo-customization elements, including Gazebo colors -->
   <xacro:include filename="$(find dji_description)/urdf/dji.gazebo" />

Commit message: changing to multiple sensors

File: dji_description/urdf/dji.xacro (robot description, xacro)
@@ -45,5 +45,5 @@
     <parent link="dji_link"/>
     <child link="hokuyo_link"/>
-    <origin xyz="0.22 0 0.4" rpy="0 0 0"/>
+    <origin xyz="0.0 0 ${height/2}" rpy="0 0 0"/>
     <axis xyz="1 0 0"/>
     <dynamics damping="1.0"/>

Commit message: fixing complication bugs after clean make. Runs on 16.04

File: dji_description/urdf/dji.xacro (robot description, xacro)
@@ -42,10 +42,9 @@
     </sensor> -->
   </link>
-  <joint name="hokuyo_joint" type="continuous">
+  <joint name="hokuyo_joint" type="fixed">
     <parent link="dji_link"/>
     <child link="hokuyo_link"/>
     <origin xyz="0.0 0 ${height/2}" rpy="0 0 0"/>
     <axis xyz="1 0 0"/>
-    <dynamics damping="1.0"/>
   </joint>
   <!-- Hokuyo Laser -->
@@ -70,51 +69,3 @@
     </inertial>
   </link>
-  <joint name="camera_joint" type="continuous">
-    <axis xyz="0 0 1" />
-    <origin xyz="0.18 0 0.2" rpy="0 0 0"/>
-    <parent link="dji_link"/>
-    <child link="camera_link"/>
-  </joint>
-  <!-- Camera -->
-  <link name="camera_link">
-    <collision>
-      <origin xyz="0 0 0" rpy="0 0 0"/>
-      <geometry>
-	<box size="0.03 0.02 0.02"/>
-      </geometry>
-    </collision>
-    <visual>
-      <origin xyz="0 0 0" rpy="0 0 0 "/>
-      <geometry>
-	    <box size="0.06 0.03 0.03"/>
-	    <!-- <cylinder length="0.06" radius="0.02"/> -->
-      </geometry>
-      <material name="white"/>
-    </visual>
-    <inertial>
-      <mass value="1e-5" />
-      <origin xyz="0 0 0" rpy="0 0 0"/>
-      <inertia ixx="1e-6" ixy="0" ixz="0" iyy="1e-6" iyz="0" izz="1e-6" />
-    </inertial>
-  </link>
-  <transmission name="tran1">
-    <type>transmission_interface/SimpleTransmission</type>
-    <joint name="hokuyo_joint">
-      <hardwareInterface>EffortJointInterface</hardwareInterface>
-    </joint>
-    <actuator name="hokuyo_motor">
-      <hardwareInterface>EffortJointInterface</hardwareInterface>
-      <mechanicalReduction>1</mechanicalReduction>
-    </actuator>
-  </transmission>
-  <transmission name="tran2">
-    <type>transmission_interface/SimpleTransmission</type>
-    <joint name="camera_joint">
-      <hardwareInterface>EffortJointInterface</hardwareInterface>
-    </joint>
-    <actuator name="camera_motor">
-      <hardwareInterface>EffortJointInterface</hardwareInterface>
-      <mechanicalReduction>1</mechanicalReduction>
-    </actuator>
-  </transmission>
 </robot>

Commit message: moving rl_manager to reactive obs. repo

File: dji_description/urdf/dji.xacro (robot description, xacro)
@@ -69,3 +69,57 @@
     </inertial>
   </link>
+  <joint name="camera_joint1" type="fixed">
+    <parent link="dji_link"/>
+    <child link="camera_link1"/>
+    <origin xyz="0.0 0 0" rpy="-1.5707963 0 -1.5707963"/>
+    <axis xyz="1 0 0"/>
+  </joint>
+  <!-- depth_cam Laser -->
+  <link name="camera_link1">
+  </link>
+  <joint name="camera_joint2" type="fixed">
+    <parent link="dji_link"/>
+    <child link="camera_link2"/>
+    <origin xyz="0.0 0 0" rpy="-1.5707963 0 -3.1415"/>
+    <axis xyz="1 0 0"/>
+  </joint>
+  <!-- depth_cam Laser -->
+  <link name="camera_link2">
+  </link>
+  <joint name="camera_joint3" type="fixed">
+    <parent link="dji_link"/>
+    <child link="camera_link3"/>
+    <origin xyz="0.0 0 0" rpy="-1.5707963 0 1.5707963"/>
+    <axis xyz="1 0 0"/>
+  </joint>
+  <!-- depth_cam Laser -->
+  <link name="camera_link3">
+  </link>
+  <joint name="camera_joint4" type="fixed">
+    <parent link="dji_link"/>
+    <child link="camera_link4"/>
+    <origin xyz="0.0 0 0" rpy="-1.5707963 0 0"/>
+    <axis xyz="1 0 0"/>
+  </joint>
+  <!-- depth_cam Laser -->
+  <link name="camera_link4">
+  </link>
+  <joint name="camera_joint5" type="fixed">
+    <parent link="dji_link"/>
+    <child link="camera_link5"/>
+    <origin xyz="0.0 0 0" rpy="0 0 -1.5707"/>
+    <axis xyz="1 0 0"/>
+  </joint>
+  <!-- depth_cam Laser -->
+  <link name="camera_link5">
+  </link>
+    <joint name="camera_joint6" type="fixed">
+    <parent link="dji_link"/>
+    <child link="camera_link6"/>
+    <origin xyz="0.0 0 0" rpy="3.141592 0 -1.5707"/>
+    <axis xyz="1 0 0"/>
+  </joint>
+  <!-- depth_cam Laser -->
+  <link name="camera_link6">
+  </link>
 </robot>

Commit message: minor parameter changes

File: dji_description/urdf/dji.xacro (robot description, xacro)
@@ -5,6 +5,6 @@
   <xacro:property name="PI" value="3.1415926535897931"/>
   <xacro:property name="mass" value="30" /> <!-- arbitrary value for mass -->
-  <xacro:property name="width" value="1.0" /> <!-- Square dimensions (widthxwidth) of beams -->
-  <xacro:property name="height" value="0.5" /> <!-- DJI height -->
+  <xacro:property name="width" value="0.01" /> <!-- Square dimensions (widthxwidth) of beams -->
+  <xacro:property name="height" value="0.01" /> <!-- DJI height -->
   <!-- Import all Gazebo-customization elements, including Gazebo colors -->
   <xacro:include filename="$(find dji_description)/urdf/dji.gazebo" />
@@ -42,31 +42,31 @@
     </sensor> -->
   </link>
-  <joint name="hokuyo_joint" type="fixed">
-    <parent link="dji_link"/>
-    <child link="hokuyo_link"/>
-    <origin xyz="0.0 0 ${height/2}" rpy="0 0 0"/>
-    <axis xyz="1 0 0"/>
-  </joint>
+  <!-- <joint name="hokuyo_joint" type="fixed"> -->
+    <!-- <parent link="dji_link"/> -->
+    <!-- <child link="hokuyo_link"/> -->
+    <!-- <origin xyz="0.0 0 ${height/2}" rpy="0 0 0"/> -->
+    <!-- <axis xyz="1 0 0"/> -->
+  <!-- </joint> -->
   <!-- Hokuyo Laser -->
-  <link name="hokuyo_link">
-    <collision>
-      <origin xyz="0 0 0.0" rpy="0 0 0"/>
-      <geometry>
-	    <box size="0.1 0.1 0.1"/>
-      </geometry>
-    </collision>
-    <visual>
-      <origin xyz="0 0 0.0" rpy="0 0 0"/>
-      <geometry>
-        <mesh filename="package://dji_description/meshes/hokuyo_utm_30lx.dae"/>
+  <!-- <link name="hokuyo_link"> -->
+    <!-- <collision> -->
+      <!-- <origin xyz="0 0 0.0" rpy="0 0 0"/> -->
+      <!-- <geometry> -->
+	    <!-- <box size="0.1 0.1 0.1"/> -->
+      <!-- </geometry> -->
+    <!-- </collision> -->
+    <!-- <visual> -->
+      <!-- <origin xyz="0 0 0.0" rpy="0 0 0"/> -->
+      <!-- <geometry> -->
+        <!-- <mesh filename="package://dji_description/meshes/hokuyo_utm_30lx.dae"/>  -->
         <!--<box size="0.1 0.1 0.1"/>-->
-      </geometry>
-    </visual>
-    <inertial>
-      <mass value="0.1" />
-      <origin xyz="0 0 0" rpy="0 0 0"/>
-      <inertia ixx="0.01" ixy="0" ixz="0" iyy="0.01" iyz="0" izz="0.01" />
-    </inertial>
-  </link>
+      <!-- </geometry> -->
+    <!-- </visual> -->
+    <!-- <inertial> -->
+      <!-- <mass value="0.1" /> -->
+      <!-- <origin xyz="0 0 0" rpy="0 0 0"/> -->
+      <!-- <inertia ixx="0.01" ixy="0" ixz="0" iyy="0.01" iyz="0" izz="0.01" /> -->
+    <!-- </inertial> -->
+  <!-- </link> -->
   <joint name="camera_joint1" type="fixed">
     <parent link="dji_link"/>

Commit message: training ddpg in sim with random env

File: dji_description/urdf/dji.xacro (robot description, xacro)
@@ -5,6 +5,6 @@
   <xacro:property name="PI" value="3.1415926535897931"/>
   <xacro:property name="mass" value="30" /> <!-- arbitrary value for mass -->
-  <xacro:property name="width" value="0.01" /> <!-- Square dimensions (widthxwidth) of beams -->
-  <xacro:property name="height" value="0.01" /> <!-- DJI height -->
+  <xacro:property name="width" value="0.2" /> <!-- Square dimensions (widthxwidth) of beams -->
+  <xacro:property name="height" value="0.2" /> <!-- DJI height -->
   <!-- Import all Gazebo-customization elements, including Gazebo colors -->
   <xacro:include filename="$(find dji_description)/urdf/dji.gazebo" />
@@ -14,5 +14,5 @@
   <link name="dji_link">
     <collision name="dji_body_collision">
-      <origin xyz="0 0 ${height/2}" rpy="0 0 0"/>
+      <origin xyz="0 0 0" rpy="0 0 0"/>
       <geometry>
 	    <box size="${width} ${width} ${height}"/>
@@ -28,5 +28,5 @@
     </visual>
     <inertial>
-      <origin xyz="0 0 ${height/2}" rpy="0 0 0"/>
+      <origin xyz="0 0 0" rpy="0 0 0"/>
       <mass value="${mass}"/>
       <inertia

Commit message: converting to laserscan

File: dji_description/urdf/dji.xacro (robot description, xacro)
@@ -42,18 +42,18 @@
     </sensor> -->
   </link>
-  <!-- <joint name="hokuyo_joint" type="fixed"> -->
-    <!-- <parent link="dji_link"/> -->
-    <!-- <child link="hokuyo_link"/> -->
-    <!-- <origin xyz="0.0 0 ${height/2}" rpy="0 0 0"/> -->
-    <!-- <axis xyz="1 0 0"/> -->
-  <!-- </joint> -->
+  <joint name="hokuyo_joint" type="fixed">
+    <parent link="dji_link"/>
+    <child link="hokuyo_link"/>
+    <origin xyz="0.0 0 ${height/2}" rpy="0 0 0"/>
+    <axis xyz="1 0 0"/>
+  </joint>
   <!-- Hokuyo Laser -->
-  <!-- <link name="hokuyo_link"> -->
-    <!-- <collision> -->
-      <!-- <origin xyz="0 0 0.0" rpy="0 0 0"/> -->
-      <!-- <geometry> -->
-	    <!-- <box size="0.1 0.1 0.1"/> -->
-      <!-- </geometry> -->
-    <!-- </collision> -->
+  <link name="hokuyo_link">
+    <collision>
+      <origin xyz="0 0 0.0" rpy="0 0 0"/>
+      <geometry>
+	    <box size="0.1 0.1 0.1"/>
+      </geometry>
+    </collision>
     <!-- <visual> -->
       <!-- <origin xyz="0 0 0.0" rpy="0 0 0"/> -->
@@ -68,58 +68,4 @@
       <!-- <inertia ixx="0.01" ixy="0" ixz="0" iyy="0.01" iyz="0" izz="0.01" /> -->
     <!-- </inertial> -->
-  <!-- </link> -->
-  <joint name="camera_joint1" type="fixed">
-    <parent link="dji_link"/>
-    <child link="camera_link1"/>
-    <origin xyz="0.0 0 0" rpy="-1.5707963 0 -1.5707963"/>
-    <axis xyz="1 0 0"/>
-  </joint>
-  <!-- depth_cam Laser -->
-  <link name="camera_link1">
-  </link>
-  <joint name="camera_joint2" type="fixed">
-    <parent link="dji_link"/>
-    <child link="camera_link2"/>
-    <origin xyz="0.0 0 0" rpy="-1.5707963 0 -3.1415"/>
-    <axis xyz="1 0 0"/>
-  </joint>
-  <!-- depth_cam Laser -->
-  <link name="camera_link2">
-  </link>
-  <joint name="camera_joint3" type="fixed">
-    <parent link="dji_link"/>
-    <child link="camera_link3"/>
-    <origin xyz="0.0 0 0" rpy="-1.5707963 0 1.5707963"/>
-    <axis xyz="1 0 0"/>
-  </joint>
-  <!-- depth_cam Laser -->
-  <link name="camera_link3">
-  </link>
-  <joint name="camera_joint4" type="fixed">
-    <parent link="dji_link"/>
-    <child link="camera_link4"/>
-    <origin xyz="0.0 0 0" rpy="-1.5707963 0 0"/>
-    <axis xyz="1 0 0"/>
-  </joint>
-  <!-- depth_cam Laser -->
-  <link name="camera_link4">
-  </link>
-  <joint name="camera_joint5" type="fixed">
-    <parent link="dji_link"/>
-    <child link="camera_link5"/>
-    <origin xyz="0.0 0 0" rpy="0 0 -1.5707"/>
-    <axis xyz="1 0 0"/>
-  </joint>
-  <!-- depth_cam Laser -->
-  <link name="camera_link5">
-  </link>
-    <joint name="camera_joint6" type="fixed">
-    <parent link="dji_link"/>
-    <child link="camera_link6"/>
-    <origin xyz="0.0 0 0" rpy="3.141592 0 -1.5707"/>
-    <axis xyz="1 0 0"/>
-  </joint>
-  <!-- depth_cam Laser -->
-  <link name="camera_link6">
   </link>
 </robot>
